File: Synapse/SNARFB-Reza/snarfb-reza_v00.sch (EAGLE design)
At the start: 8 parts

Commit message: temp stuff
Parts:
- removed LED1, LED2, LED3, LED4, LED5: WS2812, adafruit:WS2812
- added B1: (no value), rectifier:1KAB
Connections:
- removed net GND: LED1.GND, LED2.GND, LED3.GND, LED4.GND, LED5.GND
- removed net N$1: LED1.DO, LED2.DI
- removed net N$2: LED2.DO, LED3.DI
- removed net N$3: LED3.DO, LED4.DI
- removed net N$4: LED4.DO, LED5.DI
Changed lines of the file:
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@@
 <part name="GND1" library="SparkFun-Aesthetics" deviceset="GND" device=""/>
 <part name="GND2" library="SparkFun-Aesthetics" deviceset="GND" device=""/>
-<part name="GND3" library="SparkFun-Aesthetics" deviceset="GND" device=""/>
 <part name="SUPPLY4" library="SparkFun-Aesthetics" deviceset="3.3V" device=""/>
 <part name="SUPPLY5" library="SparkFun-Aesthetics" deviceset="3.3V" device=""/>
@@
 <part name="U$2" library="0_jc-custom-eagle6" deviceset="PCF2129A" device="SO20"/>
 <part name="U$3" library="0_jc-custom-eagle6" deviceset="RF100-JACK" device="JACK2"/>
-<part name="LED1" library="adafruit" deviceset="WS2812" device=""/>
-<part name="LED2" library="adafruit" deviceset="WS2812" device=""/>
-<part name="LED3" library="adafruit" deviceset="WS2812" device=""/>
-<part name="LED4" library="adafruit" deviceset="WS2812" device=""/>
-<part name="LED5" library="adafruit" deviceset="WS2812" device=""/>
+<part name="B1" library="rectifier" deviceset="1KAB" device=""/>
 </parts>
 <sheets>
@@
 <instance part="GND1" gate="1" x="10.16" y="33.02"/>
 <instance part="GND2" gate="1" x="20.32" y="33.02"/>
-<instance part="GND3" gate="1" x="274.32" y="96.52"/>
 <instance part="SUPPLY4" gate="G$1" x="53.34" y="76.2"/>
 <instance part="SUPPLY5" gate="G$1" x="60.96" y="76.2"/>
@@
 <instance part="U$2" gate="G$1" x="55.88" y="50.8"/>
 <instance part="U$3" gate="G$1" x="132.08" y="60.96"/>
-<instance part="LED1" gate="G$1" x="213.36" y="119.38"/>
-<instance part="LED2" gate="G$1" x="243.84" y="119.38"/>
-<instance part="LED3" gate="G$1" x="274.32" y="119.38"/>
-<instance part="LED4" gate="G$1" x="304.8" y="119.38"/>
-<instance part="LED5" gate="G$1" x="335.28" y="119.38"/>
+<instance part="B1" gate="1" x="35.56" y="132.08"/>
 </instances>
 <busses>
 </busses>
 <nets>
-<net name="N$1" class="0">
-<segment>
-<pinref part="LED1" gate="G$1" pin="DO"/>
-<pinref part="LED2" gate="G$1" pin="DI"/>
-<wire x1="226.06" y1="116.84" x2="231.14" y2="116.84" width="0.1524" layer="91"/>
-</segment>
-</net>
-<net name="N$2" class="0">
-<segment>
-<pinref part="LED2" gate="G$1" pin="DO"/>
-<pinref part="LED3" gate="G$1" pin="DI"/>
-<wire x1="256.54" y1="116.84" x2="261.62" y2="116.84" width="0.1524" layer="91"/>
-</segment>
-</net>
-<net name="N$3" class="0">
-<segment>
-<pinref part="LED3" gate="G$1" pin="DO"/>
-<pinref part="LED4" gate="G$1" pin="DI"/>
-<wire x1="287.02" y1="116.84" x2="292.1" y2="116.84" width="0.1524" layer="91"/>
-</segment>
-</net>
-<net name="N$4" class="0">
-<segment>
-<pinref part="LED4" gate="G$1" pin="DO"/>
-<pinref part="LED5" gate="G$1" pin="DI"/>
-<wire x1="317.5" y1="116.84" x2="322.58" y2="116.84" width="0.1524" layer="91"/>
-</segment>
-</net>
-<net name="GND" class="0">
-<segment>
-<pinref part="LED1" gate="G$1" pin="GND"/>
-<wire x1="213.36" y1="109.22" x2="213.36" y2="104.14" width="0.1524" layer="91"/>
-<wire x1="213.36" y1="104.14" x2="243.84" y2="104.14" width="0.1524" layer="91"/>
-<pinref part="LED2" gate="G$1" pin="GND"/>
-<wire x1="243.84" y1="104.14" x2="243.84" y2="109.22" width="0.1524" layer="91"/>
-<pinref part="LED3" gate="G$1" pin="GND"/>
-<wire x1="243.84" y1="104.14" x2="274.32" y2="104.14" width="0.1524" layer="91"/>
-<wire x1="274.32" y1="104.14" x2="274.32" y2="109.22" width="0.1524" layer="91"/>
-<junction x="243.84" y="104.14"/>
-<pinref part="LED4" gate="G$1" pin="GND"/>
-<wire x1="274.32" y1="104.14" x2="304.8" y2="104.14" width="0.1524" layer="91"/>
-<wire x1="304.8" y1="104.14" x2="304.8" y2="109.22" width="0.1524" layer="91"/>
-<junction x="274.32" y="104.14"/>
-<pinref part="LED5" gate="G$1" pin="GND"/>
-<wire x1="304.8" y1="104.14" x2="335.28" y2="104.14" width="0.1524" layer="91"/>
-<wire x1="335.28" y1="104.14" x2="335.28" y2="109.22" width="0.1524" layer="91"/>
-<junction x="304.8" y="104.14"/>
-<pinref part="GND3" gate="1" pin="GND"/>
-<wire x1="274.32" y1="99.06" x2="274.32" y2="104.14" width="0.1524" layer="91"/>
-</segment>
-</net>
 </nets>
 </sheet>
