File: Synapse/SNARFB-Reza/snarfbasev4a.sch (EAGLE design)
At the start: 27 parts

Commit message: computer sync
Parts:
- added BLOADER, LED8, LED9: RED, 0_jc-custom:LED0603
- added BOOT, HWB: EVQQ2, adaprog:EVQQ2
- added C10, C11, C12, C13, C14, C15, C16: 1uF, 0_jc-custom:CAP0805
- added C8, C9: 12pF, SparkFun:CAP0603-CAP
- added J1: AVR_SPI_PRG_6PTH, SparkFun:AVR_SPI_PRG_6PTH
- added LED1: red, 0_jc-custom:LED0603
- added LED10: GREEN, 0_jc-custom:LED0603
- added LED2: blue, 0_jc-custom:LED0603
- added LED3: orange, 0_jc-custom:LED0603
- added LED4: green, 0_jc-custom:LED0603
- added NX5032GA: 8MHz, adafruit:XTALNX5032
- added R10, R16, R8, R9: 220, SparkFun-Resistors:RESISTOR0805-RES
- added R11, R12, R14, R15: 1K, SparkFun-Resistors:RESISTOR0805-RES
- added R13: 10K, SparkFun-Resistors:RESISTOR0805-RES
- added R6, R7: 22, 0_jc-custom:RESISTOR0603-RES
- added SJ10: HWB, SparkFun:SOLDERJUMPERNO
- added SJ8: (no value), SparkFun:SOLDERJUMPER_2WAYPASTE2&3
- added SJ9: SOLDERJUMPERNO, SparkFun:SOLDERJUMPERNO
- added U$7: ATMEGA32U4-AU, adafruit:ATMEGA32U4-AU
- added VREG: MCP1802, 0_jc-custom:MCP1802
- added X1: USBSMD, 0_jc-custom:USBH2959CT-ND
- LM75A: device 0_jc-custom:LM75AJC-TEST -> 0_jc-custom-eagle6:LM75AJC-TEST
- R1, R2: device SparkFun:RESISTOR -> SparkFun-Resistors:RESISTOR0805-RES
- RXTX: value SERIAL_CROSSOVER -> SERIAL_CROSSOVERNORMAL; device 0_jc-custom:SERIAL_CROSSOVER -> 0_jc-custom-eagle6:SERIAL_CROSSOVERNORMAL
- VIN: value (none) -> M023.5MM; device SparkFun:M02PTH -> SparkFun-Connectors:M023.5MM
Connections:
- removed net GPIO3: RFE.GPIO3_RX_UART0, RFE.P$29, RFE.P$5
- removed net GPIO4: RFE.GPIO4_TX_UART0, RFE.P$30, RFE.P$6
- new net AREF-7: U$7.AREF
- new net HWB: HWB.P, HWB.P1, R13.1, SJ10.1, U$7.PE2(HWB)
- new net MISO: J1.1, U$7.PB3(PDO/MISO)
- new net MOSI: J1.4, U$7.PB2(PDI/MISO)
- new net MVOUT: C12.1, R11.2, SJ9.1, VREG.VOUT
- new net N$1: LED2.A, R9.2
- new net N$10: BLOADER.C, R12.1
- new net N$13: LED4.A, R16.2
- new net N$2: LED3.A, R10.2
- new net N$4: C10.2, U$7.UCAP
- new net N$5: LED9.C, R15.1
- new net N$6: LED1.A, R8.2
- new net N$8: LED10.A, R11.1
- new net N$9: LED8.C, R14.1
- new net PB4-GRN-L4: R16.1, U$7.PB4(ADC11)
- new net PB5-ORANGE-L3: R10.1, U$7.PB5(OC1A/OC4B/ADC12)
- new net PB6-BLUE-L2: R9.1, U$7.PB6(OC1B/OC4B/ADC13)
- new net PB7-RED-L1: R8.1, U$7.PB7(OC0A/OC1C/RTS)
- new net PC6-LED8: LED8.A, U$7.PC6(OC1A)
- new net PC7-LED9: LED9.A, U$7.PC7(ICP3/CLK0/OC4A)
- new net PD4: U$7.PD4(ICP1/ADC8)
- new net PD5: U$7.PD5(XCK/CTS)
- new net PD6: U$7.PD6(T1/OC4D/ADC9)
- new net PD7: U$7.PD7(OC4D/ADC10/T0)
- new net PE6-LED7-BOOTLOADER: BLOADER.A, U$7.PE6
- new net PF0-2: U$7.PF0(ADC0)
- new net PF1-3: U$7.PF1(ADC1)
- new net PF4-4: U$7.PF4(ADC4/TCK)
- new net PF5-5: U$7.PF5(ADC5/TMS)
- new net PF6-6: U$7.PF6(ADC6/TDO)
- new net PF7-7: U$7.PF7(ADC7(TDI)
- new net RST: BOOT.P, BOOT.P1, J1.5, U$7./RESET
- new net RX1: RFE.GPIO4_TX_UART0, RFE.P$30, RFE.P$6, U$7.PD3(INT3/TXD1)
- new net SCK: J1.3, U$7.PB1(SCK)
- new net SD_CS: U$7.PB0(SS)
- new net TX1: RFE.GPIO3_RX_UART0, RFE.P$29, RFE.P$5, U$7.PD2(INT2/RXD1)
- new net UD+: R6.2, U$7.D+
- new net UD-: R7.2, U$7.D-
- new net UDM: R7.1, X1.D-
- new net UDP: R6.1, X1.D+
- new net UVCC: SJ8.2, U$7.UVCC
- new net VBUS: C11.1, SJ8.1, U$7.VBUS, VREG.SHDN, VREG.VIN, X1.VBUS
- new net XTAL1: C9.2, NX5032GA.P$2, U$7.XTAL1
- new net XTAL2: C8.2, NX5032GA.P$1, U$7.XTAL2
- net GND: now also BOOT.S, BOOT.S1, C10.1, C11.2, C12.2, C13.2, C14.2, C15.2, C16.2, C8.1, C9.1, HWB.S, HWB.S1, J1.6, LED1.C, LED10.C, LED2.C, LED3.C, LED4.C, R12.2, R14.2, R15.2, SJ10.2, U$7.GND, U$7.GND1, U$7.GND2, U$7.GND3, U$7.UGND, VREG.GND, X1.GND
- net GPIO7: now also RXTX.RXD; no longer RXTX.4
- net GPIO8: now also RXTX.TXD; no longer RXTX.1
- net RXI: now also RXTX.RXF; no longer RXTX.3
- net SCL: now also U$7.PD0(INT0/OC0B)
- net SDA: now also U$7.PD1(INT1/SDA)
- net TXO: now also RXTX.TXF; no longer RXTX.2
- net VCC3: now also C13.1, C14.1, C15.1, C16.1, J1.2, R13.2, SJ8.3, SJ9.2, U$7.AVCC, U$7.AVCC1, U$7.VCC, U$7.VCC1
Other:
- note added: "15-14"
- note added: "23-24"
- note added: "35-34"
- note added: "43-44"
- note added: "ISP, Reset, and HWB Button"
- note added: "OR System Power"
- note added: "Opto-Isolate inputs Provide 4-8 outputs"
- note added: "Shows USB Power"
- note added: "Used by LUFA Status"
- note added: "When SJ5 is connected"
- note added: "and main program"
- note added: "for states or status"
- moved on the sheet: 24LC256, C1, C2, C3, C4, C5, C7, FTDI, LM75A, R1, R2, R3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

Commit message: place holder
Parts:
- added JP1: (no value), adafruit:PINHD-1X3CB
- added U$1: R7XXXDEF, 0_jc-custom-eagle6:R7XXXDEF
Connections:
- removed net 12VG: B1.-
- removed net LOW_VIN: C1.1, C3.1, VR1.SHDN, VR1.VIN, VR2.VIN
- new net VCC12: JP1.1, U$1.VOUT
- new net VCC5: C1.1, C3.1, JP1.3, VR1.SHDN, VR1.VIN, VR2.VIN
- net 12VUNREG: now also U$1.VIN
- net GND: now also B1.-, JP1.2, U$1.GND
Other:
- moved on the sheet: B1, C1, C2, C3, C4, FTDI, SJ6, SJ7, VIN, VR1, VR2

Commit message: comp sync
Parts:
- removed B1: (no value), rectifier:1KAB
- removed C11, C12, C3, C4: 1uF, 0_jc-custom:CAP0805
- removed JP1: (no value), adafruit:PINHD-1X3CB
- removed LED10: GREEN, 0_jc-custom:LED0603
- removed LED8, LED9: RED, 0_jc-custom:LED0603
- removed LM75A: LM75AJC-TEST, 0_jc-custom-eagle6:LM75AJC-TEST
- removed PCB1: PCB_DP_RECTANGLE-80X49, dp_pcb:PCB_DP_RECTANGLE-80X49
- removed R10, R16, R9: 220, SparkFun-Resistors:RESISTOR0805-RES
- removed R11, R12, R14, R15: 1K, SparkFun-Resistors:RESISTOR0805-RES
- removed RXTX: SERIAL_CROSSOVERNORMAL, 0_jc-custom-eagle6:SERIAL_CROSSOVERNORMAL
- removed SJ1, SJ2: (no value), SparkFun:SOLDERJUMPER_2WAYS
- removed SJ4, SJ5, SJ9: SOLDERJUMPERNO, SparkFun:SOLDERJUMPERNO
- removed SJ6, SJ7: (no value), SparkFun:SOLDERJUMPER_2WAYPASTE1&2
- removed SJ8: (no value), SparkFun:SOLDERJUMPER_2WAYPASTE2&3
- removed U$1: R7XXXDEF, 0_jc-custom-eagle6:R7XXXDEF
- removed VIN: M023.5MM, SparkFun-Connectors:M023.5MM
- removed VR2, VREG: MCP1802, 0_jc-custom:MCP1802
- added G1: (no value), microbuilder:BRIDGERECTIFIER
- added IC1: (no value), 0_jc-custom-eagle6:V_REG_78XXMURATA
- added J2: POWER_JACKCOMBO, SparkFun-Connectors:POWER_JACKCOMBO
- added PTC1: (no value), microbuilder:PTC1206
- added R4: 220, microbuilder:RESISTOR_4PACK
- added R5: 1K, microbuilder:RESISTOR_4PACK
- added RXLED, TXLED: yellow, 0_jc-custom:LED0603
- added U$2: M10X2, SparkFun-Connectors:M10X2
- added U1: (no value), microbuilder:NTS0102XSON8
- added U2: lm75adp, microbuilder:TEMP_LM75B
- added U3: TSL2561_DFN, microbuilder:LIGHT_TSL2561
- added USB: GREEN, 0_jc-custom:LED0603
- 2: value blue -> red
- 3: value orange -> red
- 4: value green -> red
- R3: value (none) -> 10k
- R8: value 220 -> 10K
- VR1: value MCP1802 -> MCP1826S; device 0_jc-custom:MCP1802 -> SparkFun-PowerIC:V_REG_MIC2920
- renumbered LED1 to 1, LED2 to 2, LED3 to 3, LED4 to 4, U$7 to U4
Connections:
- net UD+ renamed UD_P
- net UD- renamed UD_N
- net UDM renamed UDM_N
- net UDP renamed UDM_P
- removed net 12VUNREG: B1.+, U$1.VIN
- removed net 24VAC1: B1.AC2, VIN.1
- removed net 24VAC2: B1.AC1, VIN.2
- removed net FTDI_GND: FTDI.GND, SJ7.2
- removed net FTDI_VCC: FTDI.VCC, SJ6.2
- removed net GPIO10: RFE.GPIO10_KBI7_RTS1, RFE.P$12, RFE.P$36, SJ3.2
- removed net GPIO17: RFE.GPIO17_AD1, RFE.P$19, RFE.P$43, SJ2.3
- removed net GPIO18: RFE.GPIO18_AD0, RFE.P$20, RFE.P$44, SJ1.3
- removed net GPIO7: RFE.GPIO7_RX_UART1, RFE.P$33, RFE.P$9, RXTX.RXD
- removed net GPIO8: RFE.GPIO8_TX_UART1, RFE.P$10, RFE.P$34, RXTX.TXD
- removed net GPIO9: FTDI.CTS, RFE.GPIO9_KBI6_CTS1, RFE.P$11, RFE.P$35
- removed net MVOUT: C12.1, R11.2, SJ9.1, VREG.VOUT
- removed net N$13: 4.A, R16.2
- removed net PB4-GRN-L4: R16.1, U4.PB4(ADC11)
- removed net PB5-ORANGE-L3: R10.1, U4.PB5(OC1A/OC4B/ADC12)
- removed net PB6-BLUE-L2: R9.1, U4.PB6(OC1B/OC4B/ADC13)
- removed net PB7-RED-L1: R8.1, U4.PB7(OC0A/OC1C/RTS)
- removed net PC6-LED8: LED8.A, U4.PC6(OC1A)
- removed net PC7-LED9: LED9.A, U4.PC7(ICP3/CLK0/OC4A)
- removed net PD4: U4.PD4(ICP1/ADC8)
- removed net PD5: U4.PD5(XCK/CTS)
- removed net PD6: U4.PD6(T1/OC4D/ADC9)
- removed net PD7: U4.PD7(OC4D/ADC10/T0)
- removed net PE6-LED7-BOOTLOADER: BLOADER.A, U4.PE6
- removed net PF0-2: U4.PF0(ADC0)
- removed net PF1-3: U4.PF1(ADC1)
- removed net PF4-4: U4.PF4(ADC4/TCK)
- removed net PF5-5: U4.PF5(ADC5/TMS)
- removed net PF6-6: U4.PF6(ADC6/TDO)
- removed net PF7-7: U4.PF7(ADC7(TDI)
- removed net SCL: 24LC256.SCL, LM75A.SCL, PCF2129A.SCL, R1.1, SJ1.2, SJ4.1, U4.PD0(INT0/OC0B)
- removed net SDA: 24LC256.SDA, LM75A.SDA, PCF2129A.SDA/!CE, R2.1, SJ2.2, SJ5.1, U4.PD1(INT1/SDA)
- removed net SD_CS: U4.PB0(SS)
- removed net VCC3A: C4.1, VR2.VOUT
- new net ARXLED: RXLED.C, U4.PB0(SS)
- new net ATXLED: TXLED.C, U4.PD5(XCK/CTS)
- new net LINT: U3.INT
- new net N$12: 4.A, R4G$4.2
- new net N$3: G1.AC1, J2.PWR
- new net PB4-L4-D8: R4G$4.1, U4.PB4(ADC11)
- new net PB5-L3-D9: R4G$3.1, U4.PB5(OC1A/OC4B/ADC12)
- new net PB6-L2-D10: R4G$2.1, U4.PB6(OC1B/OC4B/ADC13)
- new net PB7-L1-D11: R4G$1.1, U4.PB7(OC0A/OC1C/RTS)
- new net PC6-D5: U$2.16, U4.PC6(OC1A)
- new net PC7-D13-LED9BLOAD: BLOADER.C, U4.PC7(ICP3/CLK0/OC4A)
- new net PD4-D4-GPIO10: RFE.GPIO10_KBI7_RTS1, RFE.P$12, RFE.P$36, U4.PD4(ICP1/ADC8)
- new net PD6-D12-I2COE: U1.OE, U4.PD6(T1/OC4D/ADC9)
- new net PD7-D6: U$2.18, U4.PD7(OC4D/ADC10/T0)
- new net PE6-D7-GPIO9: FTDI.CTS, RFE.GPIO9_KBI6_CTS1, RFE.P$11, RFE.P$35, U4.PE6
- new net PF0-A5: U$2.4, U4.PF0(ADC0)
- new net PF1-A4: U$2.6, U4.PF1(ADC1)
- new net PF4-A3: U$2.8, U4.PF4(ADC4/TCK)
- new net PF5-A2: U$2.10, U4.PF5(ADC5/TMS)
- new net PF6-A1: U$2.12, U4.PF6(ADC6/TDO)
- new net PF7-A0: U$2.14, U4.PF7(ADC7(TDI)
- new net SCL3: 24LC256.SCL, PCF2129A.SCL, R1.1, RFE.GPIO18_AD0, RFE.P$20, RFE.P$44, U1.A2, U2.SCL, U3.SCL
- new net SCL5: U1.B2, U4.PD0(INT0/OC0B)
- new net SDA3: 24LC256.SDA, PCF2129A.SDA/!CE, R2.1, RFE.GPIO17_AD1, RFE.P$19, RFE.P$43, U1.A1, U2.SDA, U3.SDA
- new net SDA5: U1.B1, U4.PD1(INT1/SDA)
- new net VBUSRAW: PTC1.2, X1.VBUS
- net GND: now also FTDI.GND, G1.-, IC1.GND, U$2.19, U$2.20, U1.GND, U2.A0, U2.A1, U2.A2, U2.GND, U3.ADDRSEL, U3.GND, USB.C; no longer B1.-, C11.2, C12.2, C3.2, C4.2, JP1.2, LED10.C, LM75A.A0, LM75A.A1, LM75A.A2, LM75A.GND, R12.2, R14.2, R15.2, SJ6.3, SJ7.1, U$1.GND, VR2.GND, VREG.GND, X1.GND
- net GPIO0: now also SJ3.2; no longer SJ5.2
- net GPIO1: now also U2.OS; no longer SJ4.2
- net GPIO11: no longer SJ1.1
- net GPIO12: no longer SJ2.1
- net GPIO13: now also U$2.15
- net GPIO14: now also U$2.13
- net GPIO15: now also U$2.9
- net GPIO16: now also U$2.11
- net GPIO2: now also U$2.3
- net GPIO5: now also U$2.5; no longer VR2.SHDN
- net GPIO6: now also U$2.7
- net N$1: now also 1.A, R4G$1.2; no longer 2.A, R9.2
- net N$10: now also R5G$4.2, USB.A; no longer BLOADER.C, R12.1
- net N$11: now also X1.GND; no longer LM75A.OS
- net N$2: now also 2.A, R4G$2.2; no longer 3.A, R10.2
- net N$5: now also BLOADER.A, R5G$1.2; no longer LED9.C, R15.1
- net N$6: now also 3.A, R4G$3.2; no longer 1.A, R8.2
- net N$7: now also G1.AC2, J2.GND, J2.GNDBREAK; no longer FTDI.DTR
- net N$8: now also R5G$2.2, TXLED.A; no longer LED10.A, R11.1
- net N$9: now also R5G$3.2, RXLED.A; no longer LED8.C, R14.1
- net RESET_L: now also FTDI.DTR
- net RST: now also R8.1
- net RXI: now also FTDI.TXO, RFE.GPIO7_RX_UART1, RFE.P$33, RFE.P$9; no longer FTDI.RXI, RXTX.RXF
- net TXO: now also FTDI.RXI, RFE.GPIO8_TX_UART1, RFE.P$10, RFE.P$34; no longer FTDI.TXO, RXTX.TXF
- net UVCC: now also U1.VCCB; no longer SJ8.2, U4.UVCC
- net VBUS: now also PTC1.1, R5G$1.1, R5G$2.1, R5G$3.1, R5G$4.1; no longer C11.1, SJ8.1, VREG.SHDN, VREG.VIN, X1.VBUS
- net VCC12: now also G1.+, IC1.IN, U$2.17; no longer JP1.1, U$1.VOUT
- net VCC3: now also FTDI.VCC, R8.2, U$2.1, U1.VCCA, U2.VCC, U3.3.3V, U4.UVCC, VR1.OUT; no longer LM75A.VCC, SJ6.1, SJ7.3, SJ8.3, SJ9.2, VR1.VOUT
- net VCC5: now also IC1.OUT, U$2.2, VR1.IN; no longer C3.1, JP1.3, VR1.SHDN, VR1.VIN, VR2.VIN
Other:
- note added: "ATMega 2x Analog Current transformer inputs"
- note added: "ATMega DS18B20 1-wire input"
- note removed: "OR System Power"
- note removed: "Shows USB Power"
- note removed: "When SJ5 is connected"
- moved on the sheet: BLOADER, C1, C13, C14, C15, C16, C2, R8

Commit message: comp sync
Parts:
- removed 1, 2, 3, 4: red, 0_jc-custom:LED0603
- removed C5: 1uF, 0_jc-custom:CAP0805
- removed C7: 10uF, 0_jc-custom:CAP0805
- removed PCF2129A: PCF2129ASO20, 0_jc-custom:PCF2129ASO20
- removed R4: 220, microbuilder:RESISTOR_4PACK
- added C21, C22, C23, C25, C34: 0.1uF, 0_jc-custom:CAP0805
- added C3: 1uF, 0_jc-custom:CAP0805
- added C4: 10uF, 0_jc-custom:CAP0805
- added RTSCTSG: (no value), SparkFun:M03PTH
- added RXTXG: RX TX G, SparkFun:M03PTH
- added U6: PCA9541SO16-2, 0_jc-custom-eagle6:PCA9541SO16-2
- added U8: MAX3232EIDWR, SparkFun:MAX232SOIC16
- J2: value POWER_JACKCOMBO -> POWER_JACKPTH; device SparkFun-Connectors:POWER_JACKCOMBO -> SparkFun-Connectors:POWER_JACKPTH
- U1: value (none) -> PCF2129ASO20; device microbuilder:NTS0102XSON8 -> 0_jc-custom:PCF2129ASO20
- renumbered 24LC256 to U5, BLOADER to BL, RXLED to RX, TXLED to TX
Connections:
- net GPIO0 renamed GPIO0_RTCINT
- net GPIO2 renamed GPIO2_PINHD
- net GPIO5 renamed GPIO5_PINHD
- net GPIO6 renamed GPIO6_PINHD
- net PC7-D13-LED9BLOAD renamed PC7-D13-LEDBL
- net XTAL1 renamed XTAL_N
- net XTAL2 renamed XTAL_P
- removed net GPIO1: RFE.GPIO1_KBI0, RFE.P$27, RFE.P$3, U2.OS
- removed net GPIO13: RFE.GPIO13_AD5, RFE.P$15, RFE.P$39, U$2.15
- removed net GPIO14: RFE.GPIO14_AD4, RFE.P$16, RFE.P$40, U$2.13
- removed net GPIO15: RFE.GPIO15_AD3, RFE.P$17, RFE.P$41, U$2.9
- removed net GPIO16: RFE.GPIO16_AD2, RFE.P$18, RFE.P$42, U$2.11
- removed net LINT: U3.INT
- removed net N$1: 1.A, R4G$1.2
- removed net N$11: X1.GND
- removed net N$12: 4.A, R4G$4.2
- removed net N$2: 2.A, R4G$2.2
- removed net N$6: 3.A, R4G$3.2
- removed net PB4-L4-D8: R4G$4.1, U4.PB4(ADC11)
- removed net PB5-L3-D9: R4G$3.1, U4.PB5(OC1A/OC4B/ADC12)
- removed net PB6-L2-D10: R4G$2.1, U4.PB6(OC1B/OC4B/ADC13)
- removed net PB7-L1-D11: R4G$1.1, U4.PB7(OC0A/OC1C/RTS)
- removed net PD4-D4-GPIO10: RFE.GPIO10_KBI7_RTS1, RFE.P$12, RFE.P$36, U4.PD4(ICP1/ADC8)
- removed net PD6-D12-I2COE: U1.OE, U4.PD6(T1/OC4D/ADC9)
- removed net PE6-D7-GPIO9: FTDI.CTS, RFE.GPIO9_KBI6_CTS1, RFE.P$11, RFE.P$35, U4.PE6
- removed net SCL5: U1.B2, U4.PD0(INT0/OC0B)
- removed net SDA5: U1.B1, U4.PD1(INT1/SDA)
- removed net UVCC: U1.VCCB
- new net !TLINT: U2.OS, U3.INT, U6.!INT_IN
- new net CTS1: RTSCTSG.2, U8.T2OUT
- new net GPIO10_PINHD: RFE.GPIO10_KBI7_RTS1, RFE.P$12, RFE.P$36, U$2.11, U8.R2OUT
- new net GPIO13_PINHD: RFE.GPIO13_AD5, RFE.P$15, RFE.P$39, U$2.13
- new net GPIO14_PINHD: RFE.GPIO14_AD4, RFE.P$16, RFE.P$40, U$2.15
- new net GPIO1_I2CINT: RFE.GPIO1_KBI0, RFE.P$27, RFE.P$3, U6.!INT0
- new net GPIO9_PINHD: RFE.GPIO9_KBI6_CTS1, RFE.P$11, RFE.P$35, U$2.9, U8.T2IN
- new net N$13: C21.2, U8.C1-
- new net N$14: C22.2, U8.C2-
- new net N$15: C34.1, U8.V+
- new net N$16: C25.1, U8.V-
- new net N$17: C21.1, U8.C1+
- new net N$18: C22.1, U8.C2+
- new net PB4-D8: U4.PB4(ADC11)
- new net PB5-D9: U4.PB5(OC1A/OC4B/ADC12)
- new net PB6-D10: U4.PB6(OC1B/OC4B/ADC13)
- new net PB7-D11-I2CRST: U4.PB7(OC0A/OC1C/RTS), U6.!RESET
- new net PD4-D4-GPIO15: RFE.GPIO15_AD3, RFE.P$17, RFE.P$41, U4.PD4(ICP1/ADC8)
- new net PD6-D12-I2C: U4.PD6(T1/OC4D/ADC9), U6.!INT1
- new net PE6-D7-GPIO16: FTDI.CTS, RFE.GPIO16_AD2, RFE.P$18, RFE.P$42, U4.PE6
- new net RTS1: RTSCTSG.3, U8.R2IN
- new net RX0: RXTXG.3, U8.R1IN
- new net SCL0: RFE.GPIO18_AD0, RFE.P$20, RFE.P$44, U6.SCL_MST0
- new net SCL1: U4.PD0(INT0/OC0B), U6.SCL_MST1
- new net SDA0: RFE.GPIO17_AD1, RFE.P$19, RFE.P$43, U6.SDA_MST0
- new net SDA1: U4.PD1(INT1/SDA), U6.SDA_MST1
- new net TX0: RXTXG.2, U8.T1OUT
- net GND: now also C23.2, C25.2, C3.1, C34.2, C4.1, RTSCTSG.1, RXTXG.1, U1.SDI, U1.VBAT, U1.VSS, U6.A0, U6.A1, U6.A2, U6.A3, U6.GND, U8.GND, X1.GND; no longer 1.C, 2.C, 3.C, 4.C, C5.1, C7.1, PCF2129A.SDI, PCF2129A.VBAT, PCF2129A.VSS, U1.GND
- net IFS: now also U1.BBS, U1.IFS; no longer PCF2129A.BBS, PCF2129A.IFS
- net R6: now also U1.!INT; no longer PCF2129A.!INT
- net RXI: now also U8.R1OUT
- net SCL3: now also U1.SCL, U6.SCL_SLAVE; no longer PCF2129A.SCL, RFE.GPIO18_AD0, RFE.P$20, RFE.P$44, U1.A2
- net SDA3: now also U1.SDA/!CE, U6.SDA_SLAVE; no longer PCF2129A.SDA/!CE, RFE.GPIO17_AD1, RFE.P$19, RFE.P$43, U1.A1
- net TXO: now also U8.T1IN
- net VCC3: now also C23.1, C3.2, C4.2, U1.VDD, U6.VCC, U8.VCC; no longer C5.2, C7.2, PCF2129A.VDD, U1.VCCA
Other:
- note added: "0xE0h read"
- note removed: "Used by LUFA Status"
- note removed: "and main program"
- note removed: "for states or status"
- moved on the sheet: C1, C2, FTDI, G1, IC1, J2, R1, R2, RFE, VR1
