File: Synapse/SNARFB-Reza/reza-connectboard.brd (EAGLE design)
At the start: 100 x 80 mm, 6 parts

Commit message: comp sync
Parts:
- removed U$2: M08X2, SparkFun-Connectors:2X8
- added U$1: M10X2, SparkFun-Connectors:2X10
Connections:
- removed net GPIO17: U$2.13
- removed net PF0-2: U$2.4
- removed net PF1-3: U$2.6
- removed net PF4-4: U$2.8
- removed net PF5-5: U$2.10
- removed net PF6-6: U$2.12
- removed net PF7-7: U$2.14
- new net GPIO13: U$1.15
- new net GPIO14: U$1.13
- new net PC6-D5: U$1.16
- new net PD7-D6: U$1.18
- new net PF0-A5: U$1.4
- new net PF1-A4: U$1.6
- new net PF4-A3: U$1.8
- new net PF5-A2: U$1.10
- new net PF6-A1: U$1.12
- new net PF7-A0: U$1.14
- new net VCC12: U$1.17
- net GND: now also U$1.19, U$1.20; no longer U$2.15, U$2.16
- net GPIO15: now also U$1.9; no longer U$2.9
- net GPIO16: now also U$1.11; no longer U$2.11
- net GPIO2: now also U$1.3; no longer U$2.3
- net GPIO5: now also U$1.5; no longer U$2.5
- net GPIO6: now also U$1.7; no longer U$2.7
- net VCC3: now also U$1.1; no longer U$2.1
- net VCC5: now also U$1.2; no longer U$2.2
Changed lines of the file:
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@@
 <class number="0" name="default" width="0.254" drill="0">
+</class>
+<class number="1" name="smallsignal" width="0.1524" drill="0">
+</class>
+<class number="2" name="Power" width="0.508" drill="0">
 </class>
 </classes>
@@
 </autorouter>
 <elements>
-<element name="U$2" library="SparkFun-Connectors" package="2X8" value="M08X2" x="6.35" y="19.05" rot="R90"/>
 <element name="JP1" library="SparkFun-Connectors" package="SCREWTERMINAL-3.5MM-2" value="M023.5MM" x="39.37" y="39.37" rot="R270"/>
 <element name="JP2" library="SparkFun-Connectors" package="SCREWTERMINAL-3.5MM-2" value="M023.5MM" x="39.37" y="16.51" rot="R270"/>
@@
 <element name="JP4" library="SparkFun-Connectors" package="SCREWTERMINAL-3.5MM-2" value="M023.5MM" x="39.37" y="24.13" rot="R270"/>
 <element name="JP5" library="SparkFun-Connectors" package="SCREWTERMINAL-3.5MM-2" value="M023.5MM" x="39.37" y="54.61" rot="R270"/>
+<element name="U$1" library="SparkFun-Connectors" package="2X10" value="M10X2" x="3.81" y="38.1" rot="R270"/>
 </elements>
 <signals>
 <signal name="GND">
-<contactref element="U$2" pad="15"/>
-<contactref element="U$2" pad="16"/>
-<wire x1="3.81" y1="36.83" x2="6.35" y2="36.83" width="0" layer="19" extent="1-1"/>
+<contactref element="U$1" pad="19"/>
+<contactref element="U$1" pad="20"/>
+<wire x1="2.54" y1="26.67" x2="5.08" y2="26.67" width="0" layer="19" extent="1-1"/>
 </signal>
 <signal name="GPIO2">
-<contactref element="U$2" pad="3"/>
+<contactref element="U$1" pad="3"/>
 </signal>
 <signal name="GPIO5">
-<contactref element="U$2" pad="5"/>
+<contactref element="U$1" pad="5"/>
 </signal>
 <signal name="GPIO6">
-<contactref element="U$2" pad="7"/>
+<contactref element="U$1" pad="7"/>
 </signal>
 <signal name="GPIO16">
-<contactref element="U$2" pad="11"/>
+<contactref element="U$1" pad="11"/>
 </signal>
 <signal name="GPIO15">
-<contactref element="U$2" pad="9"/>
+<contactref element="U$1" pad="9"/>
 </signal>
 <signal name="VCC3">
-<contactref element="U$2" pad="1"/>
-</signal>
-<signal name="PF7-7">
-<contactref element="U$2" pad="14"/>
-</signal>
-<signal name="PF4-4">
-<contactref element="U$2" pad="8"/>
-</signal>
-<signal name="PF1-3">
-<contactref element="U$2" pad="6"/>
-</signal>
-<signal name="PF0-2">
-<contactref element="U$2" pad="4"/>
-</signal>
-<signal name="PF6-6">
-<contactref element="U$2" pad="12"/>
-</signal>
-<signal name="PF5-5">
-<contactref element="U$2" pad="10"/>
+<contactref element="U$1" pad="1"/>
 </signal>
 <signal name="VCC5">
-<contactref element="U$2" pad="2"/>
-</signal>
-<signal name="GPIO17">
-<contactref element="U$2" pad="13"/>
+<contactref element="U$1" pad="2"/>
+</signal>
+<signal name="GPIO14" class="1">
+<contactref element="U$1" pad="13"/>
+</signal>
+<signal name="GPIO13" class="1">
+<contactref element="U$1" pad="15"/>
+</signal>
+<signal name="PD7-D6" class="1">
+<contactref element="U$1" pad="18"/>
+</signal>
+<signal name="PC6-D5" class="1">
+<contactref element="U$1" pad="16"/>
+</signal>
+<signal name="PF7-A0" class="1">
+<contactref element="U$1" pad="14"/>
+</signal>
+<signal name="PF4-A3" class="1">
+<contactref element="U$1" pad="8"/>
+</signal>
+<signal name="PF1-A4" class="1">
+<contactref element="U$1" pad="6"/>
+</signal>
+<signal name="PF0-A5" class="1">
+<contactref element="U$1" pad="4"/>
+</signal>
+<signal name="PF6-A1" class="1">
+<contactref element="U$1" pad="12"/>
+</signal>
+<signal name="PF5-A2" class="1">
+<contactref element="U$1" pad="10"/>
+</signal>
+<signal name="VCC12" class="2">
+<contactref element="U$1" pad="17"/>
 </signal>
 </signals>

Commit message: sync
Parts:
- added JP11, JP6, JP8, JP9: (no value), SparkFun-Connectors:SCREWTERMINAL-3.5MM-3
- added JP12, JP13, JP14, JP15, JP16, JP17, JPPIR: M023.5MM, SparkFun-Connectors:SCREWTERMINAL-3.5MM-2
- added R1: (no value), adafruit:0805-THM
- added RELAY_MEGA, RELAY_RFE: (no value), SparkFun-Connectors:1X06
- added U$2: (no value), 0_jc-custom-eagle6:ENVIOSYS_LOGO2
- JP3: value M023.5MM -> (none); device SparkFun-Connectors:SCREWTERMINAL-3.5MM-2 -> SparkFun-Connectors:SCREWTERMINAL-3.5MM-3
- moved U$1 65.2 mm to (68.6, 30.5)
- moved JP5 54.6 mm to (16.5, 5.08), turned to 180 degrees
- moved JP1 43.4 mm to (66.0, 5.08), turned to 180 degrees
- moved JP2 30.6 mm to (8.89, 19.1), turned to 90 degrees
- moved JP4 23.6 mm to (25.4, 5.08), turned to 180 degrees
- moved JP3 16.9 mm to (22.9, 43.2), turned to 0 degrees
Connections:
- net GND: now also JP1.1, JP11.1, JP12.1, JP13.1, JP14.1, JP15.1, JP16.1, JP17.1, JP2.1, JP6.1, JP9.1, RELAY_MEGA.1, RELAY_RFE.1
- net GPIO13: now also JP4.2
- net GPIO14: now also JP4.1
- net GPIO15: now also JP6.2, RELAY_RFE.2
- net GPIO16: now also JP11.2
- net GPIO2: now also JP3.2, RELAY_RFE.5
- net GPIO5: now also JP3.1, RELAY_RFE.4
- net GPIO6: now also JP6.3, RELAY_RFE.3
- net PC6-D5: now also JPPIR.1
- net PD7-D6: now also JP1.2, R1.2
- net PF0-A5: now also JP9.2, RELAY_MEGA.2
- net PF1-A4: now also JP9.3, RELAY_MEGA.3
- net PF4-A3: now also JP8.1, RELAY_MEGA.4
- net PF5-A2: now also JP8.2, RELAY_MEGA.5
- net PF6-A1: now also JP5.2
- net PF7-A0: now also JP5.1
- net VCC12: now also JP12.2, JP13.2, JP2.2
- net VCC3: now also JP11.3, JP16.2, JP17.2, JPPIR.2, R1.1
- net VCC5: now also JP14.2, JP15.2, JP3.3, JP8.3, RELAY_MEGA.6, RELAY_RFE.6
Routing:
- net GND: track 0.00 -> 163.8 mm
- net VCC3: track 0.00 -> 92.6 mm
- net VCC12: track 0.00 -> 84.3 mm
- net PF6-A1: track 0.00 -> 83.3 mm
- net VCC5: track 0.00 -> 79.7 mm
- net PF7-A0: track 0.00 -> 78.2 mm
- net GPIO14: track 0.00 -> 74.0 mm
- net GPIO15: track 0.00 -> 60.4 mm
- net GPIO6: track 0.00 -> 56.5 mm
- net GPIO13: track 0.00 -> 53.3 mm
- net GPIO5: track 0.00 -> 52.0 mm
- net GPIO2: track 0.00 -> 50.5 mm
- net PF0-A5: track 0.00 -> 45.0 mm
- net PF1-A4: track 0.00 -> 44.9 mm
- net PC6-D5: track 0.00 -> 43.9 mm
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- added copper zone on layer 16, net N$1
- added copper zone on layer 1, net N$2
Other:
- board size 100 x 80 mm -> 72.1 x 48.2 mm
- board text added: "1"
- board text added: "1-Wire"
- board text added: "12"
- board text added: "2"
- board text added: "3"
- board text added: "4"
- board text added: "A0"
- board text added: "A1"
- board text added: "G"
- board text added: "GND"
- board text added: "IO13"
- board text added: "IO14"
- board text added: "IO16"
- board text added: "PIR"
- board text added: "R"
- board text added: "V"
- board text added: "V12"
- board text added: "V3"
- board text added: "V5"
